File: PSUExtensionBoard/PSUExtensionBoard.sch (KiCad schematic (older format))
At the start: 14 parts

Commit message: Changed Ext Board to add 5V, CV, Gate
Parts:
- removed J_OUT10, J_OUT2, J_OUT3, J_OUT4, J_OUT5, J_OUT6, J_OUT7, J_OUT8, J_OUT9: Conn_02x05_Odd_Even, Connector_PinHeader_2.54mm:PinHeader_2x05_P2.54mm_Vertical, symbol Connector_Generic:Conn_02x05_Odd_Even
- added C1: 220nF, Capacitor_SMD:C_0805_2012Metric_Pad1.15x1.40mm_HandSolder, symbol Device:C
- added C2: 100nF, Capacitor_SMD:C_0805_2012Metric_Pad1.15x1.40mm_HandSolder, symbol Device:C
- added D_5VPP1: LED, LED_SMD:LED_0805_2012Metric_Pad1.15x1.40mm_HandSolder, symbol Device:LED
- added J_OUT1, J_OUT2, J_OUT3, J_OUT4, J_OUT5, J_OUT6, J_OUT7, J_OUT8: Conn_02x08_Odd_Even, Connector_PinHeader_2.54mm:PinHeader_2x08_P2.54mm_Vertical, symbol Connector_Generic:Conn_02x08_Odd_Even
- added R_5VPP1: 2K7, Resistor_SMD:R_0805_2012Metric_Pad1.15x1.40mm_HandSolder, symbol Device:R
- added U_REG1: L7805, Package_TO_SOT_SMD:TO-263-3_TabPin2, symbol Regulator_Linear:L7805
- D_NEG1, D_POS1: footprint LED_THT:LED_D5.0mm -> LED_SMD:LED_0805_2012Metric_Pad1.15x1.40mm_HandSolder
- R_NEG1, R_POS1: value 1K -> 2K7; footprint Resistor_THT:R_Axial_DIN0207_L6.3mm_D2.5mm_P7.62mm_Horizontal -> Resistor_SMD:R_0805_2012Metric_Pad1.15x1.40mm_HandSolder
- renumbered J_OUT1 to J_IN1
Connections:
- net labels added: -12V, 12V, 5V, CV, GATE
- wire segments 222 -> 199

Commit message: Created SMT version of AdjustablePSU, RevB
Parts:
- D_5VPP1, D_NEG1, D_POS1: MouserNo (none) -> 630-HSMS-C150
- R_5VPP1, R_NEG1, R_POS1: MouserNo (none) -> 71-CRCW08052K70JNE
- U_REG1: MouserNo (none) -> 511-L7805CD2T-TR
Changed lines of the file:
@@
 EESchema Schematic File Version 4
-LIBS:PSUExtensionBoard-cache
 EELAYER 26 0
 EELAYER END
@@
 F 2 "LED_SMD:LED_0805_2012Metric_Pad1.15x1.40mm_HandSolder" H 800 5200 50  0001 C CNN
 F 3 "~" H 800 5200 50  0001 C CNN
+F 4 "630-HSMS-C150" H 800 5200 50  0001 C CNN "MouserNo"
 	1    800  5200
 	0    1    -1   0
@@
 F 2 "LED_SMD:LED_0805_2012Metric_Pad1.15x1.40mm_HandSolder" H 3700 5200 50  0001 C CNN
 F 3 "~" H 3700 5200 50  0001 C CNN
+F 4 "630-HSMS-C150" H 3700 5200 50  0001 C CNN "MouserNo"
 	1    3700 5200
 	0    1    1    0
@@
 F 2 "Resistor_SMD:R_0805_2012Metric_Pad1.15x1.40mm_HandSolder" V 3630 4700 50  0001 C CNN
 F 3 "~" H 3700 4700 50  0001 C CNN
+F 4 "71-CRCW08052K70JNE" H 3700 4700 50  0001 C CNN "MouserNo"
 	1    3700 4700
 	-1   0    0    1
@@
 F 2 "Resistor_SMD:R_0805_2012Metric_Pad1.15x1.40mm_HandSolder" V 730 4700 50  0001 C CNN
 F 3 "~" H 800 4700 50  0001 C CNN
+F 4 "71-CRCW08052K70JNE" H 800 4700 50  0001 C CNN "MouserNo"
 	1    800  4700
 	-1   0    0    -1
@@
 F 2 "Package_TO_SOT_SMD:TO-263-3_TabPin2" H 1600 1500 50  0001 L CIN
 F 3 "http://www.st.com/content/ccc/resource/technical/document/datasheet/41/4f/b3/b0/12/d4/47/88/CD00000444.pdf/files/CD00000444.pdf/jcr:content/translations/en.CD00000444.pdf" H 1575 1600 50  0001 C CNN
+F 4 "511-L7805CD2T-TR" H 1575 1650 50  0001 C CNN "MouserNo"
 	1    1575 1650
 	1    0    0    -1
@@
 F 2 "Resistor_SMD:R_0805_2012Metric_Pad1.15x1.40mm_HandSolder" V 2680 1650 50  0001 C CNN
 F 3 "~" H 2750 1650 50  0001 C CNN
+F 4 "71-CRCW08052K70JNE" H 2750 1650 50  0001 C CNN "MouserNo"
 	1    2750 1650
 	0    1    1    0
@@
 F 2 "LED_SMD:LED_0805_2012Metric_Pad1.15x1.40mm_HandSolder" H 3300 1650 50  0001 C CNN
 F 3 "~" H 3300 1650 50  0001 C CNN
+F 4 "630-HSMS-C150" H 3300 1650 50  0001 C CNN "MouserNo"
 	1    3300 1650
 	-1   0    0    1
