File: FixedPSU/FixedPSU.kicad_pcb (KiCad board)
At the start: 2 copper layers, 88.9 x 68.6 mm, 32 parts

Commit message: added gerbers files for fixed psu and extension board
Parts:
- turned D_POS1 to 180 degrees
Routing:
- net GND: track 377.5 -> 0.06 mm
- net /AC_IN: track 38.1 -> 34.5 mm
- net /DC_POS_IN: track 179.6 -> 181.4 mm
- added copper zone on B.Cu, net GND
Other:
- board text added: "+12VDC 1400mA -12VDC 1400mA (POLARITY MARKED)"
- board text added: "12VAC INPUT"
- board text removed: "+12VDC 1400mA -12VDC 1400mA (MARKED)"
- board text removed: "AC INPUT ONLY!"
